Commit message: fixes

File: src/slamify/description/imu.xacro (robot description, xacro)
@@ -28,9 +28,45 @@
         </xacro:inertial_box>
     </link>
+    <joint name="joint_name" type="fixed">
+        <parent link="imu_frame" />
+        <child link="mag_link" />
+    </joint>
+    <link name="mag_link" />
+    <gazebo reference="mag_link">
+        <!-- <sensor name="magnetometer" type="magnetometer">
+            <always_on>true</always_on>
+            <update_rate>200</update_rate>
+            <magnetometer>
+                <x>
+                    <noise type="gaussian">
+                        <mean>0.0</mean>
+                        <stddev>0.001</stddev>
+                    </noise>
+                </x>
+                <y>
+                    <noise type="gaussian">
+                        <mean>0.0</mean>
+                        <stddev>0.001</stddev>
+                    </noise>
+                </y>
+                <z>
+                    <noise type="gaussian">
+                        <mean>0.0</mean>
+                        <stddev>0.001</stddev>
+                    </noise>
+                </z>
+            </magnetometer>
+            <plugin name="mag" filename="libgazebo_ros_magnetometer.so">
+                <ros>
+                    <remapping>~/out:=magnetometer/data</remapping>
+                </ros>
+            </plugin>
+        </sensor> -->
+    </gazebo>
     <gazebo reference="imu_frame">
         <initial_orientation_as_reference>false</initial_orientation_as_reference>
         <material>Gazebo/Green</material>
         <gravity>true</gravity>
-        <sensor name="tb3_imu" type="imu">
+        <sensor name="imu" type="imu">
         <always_on>true</always_on>
         <update_rate>200</update_rate>
@@ -79,6 +115,5 @@
         <plugin name="imu_sensor" filename="libgazebo_ros_imu_sensor.so">
           <ros>
-            <!-- <namespace>/tb3</namespace> -->
-            <remapping>~/out:=imu_raw</remapping>
+            <remapping>~/out:=imu</remapping>
           </ros>
         </plugin>
@@ -86,5 +121,2 @@
     </gazebo>
 </robot>
-<!--
-    <link name="imu_link">
-    </link> -->

File: src/slamify/description/robot.urdf.xacro (robot description, xacro)
@@ -6,19 +6,18 @@
     <!-- lidar -->
     <xacro:include filename="lidar.xacro" />
-    <!-- imu -->
+    <!-- imu + magnetometer-->
     <xacro:include filename="imu.xacro" />
-    <!-- magnetometer -->
-    <xacro:include filename="magnetometer.xacro" />
-    <!-- camera -->
+    <!-- camera (light weight and easy)-->
     <xacro:include filename="camera.xacro" />
-    <!-- depth cam -->
-    <xacro:include filename="depth_camera.xacro" />
+            <!-- enable only 1 -->
+    <!-- depth cam  (computationally heavy)-->
+    <!-- <xacro:include filename="depth_camera.xacro" /> -->
     <!-- multiple cam -->
-    <xacro:include filename="multi_camera.xacro" />
+    <!-- <xacro:include filename="multi_camera.xacro" /> -->
     <!-- gps -->
-    <xacro:include filename="gps.xacro" />
+    <!-- <xacro:include filename="gps.xacro" /> -->
     <!-- bumper -->
-    <xacro:include filename="bumper.xacro" />
+    <!-- <xacro:include filename="bumper.xacro" /> -->
     <!-- display video -->
-    <xacro:include filename="disp_video.xacro" />
+    <!-- <xacro:include filename="disp_video.xacro" /> -->
 </robot>
